File: From Programmer's Reference Guide/C64.sch (EAGLE design)
At the start: 239 parts, among them CN2 USERPORT-C64-EDGE, CN3 CASSETTEPORT, CN4 MAB6H, CN5 MAB8SH, CN6 EXPANSIONPORT, CN7 MAB7SH, Q1 tp29b, Q2 2N4401, Q3 2N3904, Q4 2N2222, Q5 2N2222, Q6 2N2222, Q7 2N2222, Q8 2N2222, SW1 9077-2, U1 6526, U10 4164, U11 4164, U12 4164, U13 74LS257N, U14 74LS258N, U15 74LS139N, U16 4066, U17 C64PLA, U18 6581, U19 6569, U2 6526, U20 556DIGITAL, U21 4164, U22 4164, U23 4164, U24 4164, U25 74LS257N, U26 74LS373N, U27 74LS08N, U28 4066, U29 74LS74N, U3 2364, U30 74LS193N, U31 74629, U32 MC4044, U4 2364, U5 2332, U6 2114, U7 6510, U8 7406N, U9 4164, Y1 17.73 MHz

Commit message: Cleaned up schematic
Also corrected values to those written on schematic. Added link to BOM
Parts:
- C5: value 0.47uF -> 0.47 uF
- C58, C98, C99: value 0.1uF -> 0.1 uF
- R16, R23, R28, R29, R30, R31, R36, R4: value 1K -> 1 K
- R19: value 15K -> 15 K
- R3, R7: value 10K -> 10 K
- R34: value 47K -> 47 K
- R35: value 470K -> 470 K
- R41, R50: value 1M -> 1 M
Other:
- note added: "Commodore C64 Rev A Replica Schematic Based on schematic done by Ruud Baltissen. Values and footprints corrected by Bo Herrmannsen"
Changed lines of the file:
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@@
 <part name="V2" library="supply2" deviceset="VCC" device=""/>
 <part name="V9" library="supply2" deviceset="+12V" device=""/>
-<part name="R7" library="rcl" deviceset="R-EU_" device="0204/2V" value="10K"/>
+<part name="R7" library="rcl" deviceset="R-EU_" device="0204/2V" value="10 K"/>
 <part name="C37" library="rcl" deviceset="C-EU" device="075-032X103" value="1000 pF"/>
 <part name="GND1" library="supply1" deviceset="GND" device=""/>
@@
 <part name="C20" library="rcl" deviceset="C-EU" device="075-032X103" value="0.22 uF 100V"/>
 <part name="C21" library="rcl" deviceset="C-EU" device="075-032X103" value="0.22 uF 100V"/>
-<part name="C98" library="rcl" deviceset="C-EU" device="075-032X103" value="0.1uF"/>
-<part name="C99" library="rcl" deviceset="C-EU" device="075-032X103" value="0.1uF"/>
+<part name="C98" library="rcl" deviceset="C-EU" device="075-032X103" value="0.1 uF"/>
+<part name="C99" library="rcl" deviceset="C-EU" device="075-032X103" value="0.1 uF"/>
 <part name="GND23" library="supply1" deviceset="GND" device=""/>
 <part name="GND24" library="supply1" deviceset="GND" device=""/>
@@
 <part name="U8" library="74xx-us" deviceset="74*06" device="N"/>
 <part name="GND59" library="supply1" deviceset="GND" device=""/>
-<part name="R34" library="rcl" deviceset="R-EU_" device="0204/2V" value="47K"/>
+<part name="R34" library="rcl" deviceset="R-EU_" device="0204/2V" value="47 K"/>
 <part name="U20" library="0RB_Lineair" deviceset="556DIGITAL" device=""/>
 <part name="C24" library="rcl" deviceset="CPOL-EU" device="E3.5-10" value="10 uF 25V"/>
-<part name="R50" library="rcl" deviceset="R-EU_" device="0204/2V" value="1M"/>
+<part name="R50" library="rcl" deviceset="R-EU_" device="0204/2V" value="1 M"/>
 <part name="C105" library="rcl" deviceset="C-EU" device="075-032X103" value="0.1 uF"/>
 <part name="GND60" library="supply1" deviceset="GND" device=""/>
@@
 <part name="GND61" library="supply1" deviceset="GND" device=""/>
 <part name="R33" library="rcl" deviceset="R-EU_" device="0204/2V" value="47K"/>
-<part name="R41" library="rcl" deviceset="R-EU_" device="0204/2V" value="1M"/>
+<part name="R41" library="rcl" deviceset="R-EU_" device="0204/2V" value="1 M"/>
 <part name="C38" library="rcl" deviceset="C-EU" device="075-032X103" value="51 pF"/>
 <part name="GND62" library="supply1" deviceset="GND" device=""/>
 <part name="C23" library="rcl" deviceset="C-EU" device="075-032X103" value="360 pF"/>
-<part name="R35" library="rcl" deviceset="R-EU_" device="0204/2V" value="470K"/>
+<part name="R35" library="rcl" deviceset="R-EU_" device="0204/2V" value="470 K"/>
 <part name="GND63" library="supply1" deviceset="GND" device=""/>
 <part name="R26" library="rcl" deviceset="R-EU_" device="0204/2V" value="75"/>
 <part name="R27" library="pot" deviceset="TRIM_EU-" device="CA6H" value="2 K Trim Pot"/>
 <part name="V18" library="supply2" deviceset="+5V/2" device="" value="+5Vc"/>
-<part name="C58" library="rcl" deviceset="C-EU" device="075-032X103" value="0.1uF"/>
+<part name="C58" library="rcl" deviceset="C-EU" device="075-032X103" value="0.1 uF"/>
 <part name="FB16" library="0RB_Passive" deviceset="FERRIT" device=""/>
 <part name="Y1" library="crystal" deviceset="HC49TL-H" device="" value="17.73 MHz"/>
@@
 <part name="V21" library="supply2" deviceset="+5V/2" device="" value="+5Vc"/>
 <part name="U31" library="0RB_TTL" deviceset="74629" device=""/>
-<part name="R23" library="rcl" deviceset="R-EU_" device="0204/2V" value="1K"/>
+<part name="R23" library="rcl" deviceset="R-EU_" device="0204/2V" value="1 K"/>
 <part name="R22" library="rcl" deviceset="R-EU_" device="0204/2V" value="1.5 K"/>
 <part name="C87" library="rcl" deviceset="C-EU" device="075-032X103" value="0.1 uF"/>
@@
 <part name="C86" library="rcl" deviceset="C-EU" device="075-032X103" value="39 pF 50V 5%"/>
 <part name="Q7" library="transistor-small-signal" deviceset="2N2222" device=""/>
-<part name="R19" library="rcl" deviceset="R-EU_" device="0204/2V" value="15K"/>
+<part name="R19" library="rcl" deviceset="R-EU_" device="0204/2V" value="15 K"/>
 <part name="C85" library="rcl" deviceset="C-EU" device="075-032X103" value="0.47 uF"/>
 <part name="R17" library="rcl" deviceset="R-EU_" device="0204/2V" value="1.2 K"/>
-<part name="R16" library="rcl" deviceset="R-EU_" device="0204/2V" value="1K"/>
+<part name="R16" library="rcl" deviceset="R-EU_" device="0204/2V" value="1 K"/>
 <part name="C84" library="rcl" deviceset="C-EU" device="075-032X103" value="0.1 uF"/>
 <part name="GND67" library="supply1" deviceset="GND" device=""/>
@@
 <part name="GND68" library="supply1" deviceset="GND" device=""/>
 <part name="C36" library="rcl" deviceset="C-EU" device="075-032X103" value="20 pF 50V"/>
-<part name="R31" library="rcl" deviceset="R-EU_" device="0204/2V" value="1K"/>
+<part name="R31" library="rcl" deviceset="R-EU_" device="0204/2V" value="1 K"/>
 <part name="V23" library="supply2" deviceset="VCC" device=""/>
 <part name="U3" library="0RB_Memory" deviceset="2364" device=""/>
@@
 <part name="FB7" library="0RB_Passive" deviceset="FERRIT" device=""/>
 <part name="FB9" library="0RB_Passive" deviceset="FERRIT" device=""/>
-<part name="R29" library="rcl" deviceset="R-EU_" device="0204/2V" value="1K"/>
-<part name="R30" library="rcl" deviceset="R-EU_" device="0204/2V" value="1K"/>
-<part name="R28" library="rcl" deviceset="R-EU_" device="0204/2V" value="1K"/>
+<part name="R29" library="rcl" deviceset="R-EU_" device="0204/2V" value="1 K"/>
+<part name="R30" library="rcl" deviceset="R-EU_" device="0204/2V" value="1 K"/>
+<part name="R28" library="rcl" deviceset="R-EU_" device="0204/2V" value="1 K"/>
 <part name="V26" library="supply2" deviceset="VCC" device=""/>
 <part name="CN2" library="0RB_Commodore" deviceset="USERPORT-C64-EDGE" device=""/>
@@
 <part name="R2" library="rcl" deviceset="R-EU_" device="0204/2V" value="1.5 K"/>
 <part name="V30" library="supply2" deviceset="+9V" device=""/>
-<part name="R3" library="rcl" deviceset="R-EU_" device="0204/2V" value="10K"/>
+<part name="R3" library="rcl" deviceset="R-EU_" device="0204/2V" value="10 K"/>
 <part name="GND78" library="supply1" deviceset="GND" device=""/>
 <part name="GND79" library="supply1" deviceset="GND" device=""/>
-<part name="R4" library="rcl" deviceset="R-EU_" device="0204/2V" value="1K"/>
+<part name="R4" library="rcl" deviceset="R-EU_" device="0204/2V" value="1 K"/>
 <part name="V31" library="supply2" deviceset="VCC" device=""/>
 <part name="GND80" library="supply1" deviceset="GND" device=""/>
 <part name="CN6" library="0RB_Commodore" deviceset="EXPANSIONPORT-C64" device="" value="EXPANSIONPORT"/>
 <part name="RP3" library="0RB_Passive" deviceset="RP8" device="" value="3.3 K"/>
-<part name="R36" library="rcl" deviceset="R-EU_" device="0204/2V" value="1K"/>
+<part name="R36" library="rcl" deviceset="R-EU_" device="0204/2V" value="1 K"/>
 <part name="V32" library="supply2" deviceset="VCC" device=""/>
 <part name="V34" library="supply2" deviceset="VCC" device=""/>
@@
 <part name="V54" library="supply2" deviceset="VCC" device=""/>
 <part name="GND103" library="supply1" deviceset="GND" device=""/>
-<part name="C5" library="rcl" deviceset="C-EU" device="075-032X103" value="0.47uF"/>
+<part name="C5" library="rcl" deviceset="C-EU" device="075-032X103" value="0.47 uF"/>
 <part name="V55" library="supply2" deviceset="VCC" device=""/>
 <part name="GND104" library="supply1" deviceset="GND" device=""/>
@@
 <part name="GND115" library="supply1" deviceset="GND" device=""/>
 <part name="C68" library="rcl" deviceset="C-EU" device="075-032X103" value="0.1 uF"/>
+<part name="FRAME1" library="frames" deviceset="FRAME_D_L" device=""/>
 </parts>
 <sheets>
 <sheet>
 <plain>
+<text x="104.14" y="-195.58" size="1.778" layer="94">Commodore C64 Rev A Replica Schematic
+Based on schematic done by Ruud Baltissen.
+Values and footprints corrected by Bo Herrmannsen</text>
 </plain>
 <instances>
@@
 <instance part="C68" gate="G$1" x="101.6" y="289.56"/>
 <instance part="RP4" gate="B" x="-50.8" y="208.28"/>
+<instance part="FRAME1" gate="G$1" x="-223.52" y="-220.98"/>
+<instance part="FRAME1" gate="G$2" x="101.6" y="-220.98"/>
 </instances>
 <busses>
@@
 </schematic>
 </drawing>
+<compatibility>
+<note version="6.3" minversion="6.2.2" severity="warning">
+Since Version 6.2.2 text objects can contain more than one line,
+which will not be processed correctly with this version.
+</note>
+</compatibility>
 </eagle>
